File: lab4_audio/kiCAD/lab4_audio_schematic/lab4_audio_schematic.kicad_sch (KiCad schematic)
At the start: 0 parts

Commit message: Cleaning up code from a couple different labs
For redos
Parts:
- added C3: 220u, symbol Device:C
- added C4: 47n, symbol Device:C
- added J1: NUCLEO-L432KC, symbol Connector_Generic:Conn_01x04
- added LS1: Speaker, symbol Device:Speaker
- added R1: 10, symbol Device:R
- added RV1: 100, symbol Device:R_Potentiometer
- added U1: LM386, symbol Amplifier_Audio:LM386
Connections:
- new net: C3.1, C4.2, U1.5
- new net: C3.2, LS1.1
- new net: J1.PA6 (GPIOA), RV1.1
- new net: C4.1, R1.1
- new net: RV1.2, U1.3 (+)
- new net +5V: J1.5V, U1.6 (V+)
- new net GND: J1.GND, LS1.2, R1.2, RV1.3, U1.2 (-), U1.4 (GND)
- no-connect marks 0 -> 3
Other:
- note added: "1 1"
- note added: "10/27/2025"
- note added: "Lucas Lemos"
- note added: "PWM Audio Lab"
